Commit message: urdf fix two

File: hopper_sim/hopper.urdf (robot description, URDF)
Before this commit: robot hopper, 5 links, 2 joints
Links:
- removed link knee
- removed link leg2
Joints:
- removed joint leg2_knee_joint

Commit message: urdf fix two

File: hopper_sim/hopper.urdf (robot description, URDF)
Before this commit: robot hopper, 3 links, 1 joints
Links:
- removed link hip
- removed link leg1
Joints:
- removed joint leg1_hip_joint
