Commit message: urdf fix two

File: hopper_sim/urdf/hopper.urdf (robot description, URDF)
Before this commit: robot hopper, 0 links, 0 joints
Links:
- added link head, mass 100; collision box size=1 1 1; visual box size=1 1 1
- added link hip, mass 1; collision sphere radius=0.1; visual sphere radius=0.1
- added link knee, mass 1; collision sphere radius=0.1; visual sphere radius=0.1
- added link leg1, mass 10; collision cylinder length=1 radius=0.1; visual cylinder length=1 radius=0.1
- added link leg2, mass 10; collision cylinder length=1 radius=0.1; visual cylinder length=1 radius=0.1
Joints:
- added joint leg1_hip_joint: type fixed, parent leg1, child hip
- added joint leg2_knee_joint: type fixed, parent leg2, child knee

Commit message: urdf fix two

File: hopper_sim/urdf/hopper.urdf (robot description, URDF)
Before this commit: robot hopper, 5 links, 2 joints
Joints:
- joint leg1_hip_joint: child hip -> leg1; parent leg1 -> hip
- joint leg2_knee_joint: child knee -> leg2; parent leg2 -> knee

Commit message: urdf fix two

File: hopper_sim/urdf/hopper.urdf (robot description, URDF)
Before this commit: robot hopper, 7 links, 3 joints
Joints:
- added joint head_leg1_joint1: type revolute, parent head, child hip, axis 1 0 0, limit lower=-0.78539 upper=0.78539 effort=30 velocity=30
- added joint head_leg1_joint2: type revolute, parent head, child hip, axis 0 0 1, limit lower=-0.78539 upper=0.78539 effort=30 velocity=30
- added joint leg1_leg2_joint: type revolute, parent leg1, child knee, axis 1 0 0, limit lower=-0.78539 upper=0.78539 effort=30 velocity=30
- added joint leg2_foot_joint: type revolute, parent leg2, child ankle, axis 0 0 1, limit lower=-0.78539 upper=0.78539 effort=30 velocity=30

Commit message: urdf fix two

File: hopper_sim/urdf/hopper.urdf (robot description, URDF)
Before this commit: robot hopper, 7 links, 7 joints
Joints:
- removed joint leg2_foot_joint
- added joint leg2_foot_joint1: type revolute, parent leg2, child ankle, axis 1 0 0, limit lower=-0.78539 upper=0.78539 effort=30 velocity=30
- added joint leg2_foot_joint2: type revolute, parent leg2, child ankle, axis 0 0 1, limit lower=-0.78539 upper=0.78539 effort=30 velocity=30

Commit message: urdf fix two

File: hopper_sim/urdf/hopper.urdf (robot description, URDF)
Before this commit: robot hopper, 7 links, 8 joints
Joints:
- joint foot_ankle_joint: child ankle -> foot; parent foot -> ankle
